Commit message: made code more modifiable and also added and option for adding obstacles in hover

File: gym_pybullet_drones/assets/architrave.urdf (robot description, URDF)
Before this commit: robot architrave, 1 links, 0 joints
Links:
- link base_link: geometry collision box size=.8 .12 .05; visual box size=.8 .12 .05
